Commit message: Working urdf model

File: crio_driver/urdf/robot.urdf (robot description, URDF)
Before this commit: robot test_robot, 5 links, 4 joints
Links:
- link base_link: geometry collision box size=0.16 0.16 0.12; visual box size=0.16 0.16 0.12
- link lwheel: geometry collision cylinder length=0.008 radius=0.046; visual cylinder length=0.008 radius=0.046
- link rwheel: geometry collision cylinder length=0.008 radius=0.046; visual cylinder length=0.008 radius=0.046
